Commit message: fix controller

File: fra333_lab4_01/fra333_lab4_01_description/robot/ros2controller_gazebo.xacro (robot description, xacro)
@@ -15,5 +15,5 @@
     <!-- This plugin will publish the joint_states for the selected joints
             (which robot_state_publisher can then use to broadcast the approprate tf). -->
-    <gazebo>
+    <!-- <gazebo>
         <plugin name="gazebo_ros_joint_state_publisher"
             filename="libgazebo_ros_joint_state_publisher.so">
@@ -23,5 +23,5 @@
             <joint_name>link_2_to_3</joint_name>
         </plugin>
-    </gazebo>
+    </gazebo> -->
     <!-- This plugin will read a JointTrajectory message from the /set_joint_trajectory topic
             and move the machine accordingly. It's a bit clunky but it works. -->
@@ -111,5 +111,5 @@
     <gazebo>
         <plugin name="gazebo_ros2_control" filename="libgazebo_ros2_control.so">
-            <parameters>$(find fra333_lab3_01_description)/config/sentinel_controller.yaml</parameters>
+            <parameters>$(find fra333_lab4_01_description)/config/sentinel_controller.yaml</parameters>
         </plugin>
     </gazebo>

File: fra333_lab4_01/fra333_lab4_01_description/robot/sentinel.urdf.xacro (robot description, xacro)
@@ -6,5 +6,5 @@
         <visual>
             <geometry>
-                <mesh filename="file:///$(find fra333_lab3_01_description)/mesh/link_0.STL"/>
+                <mesh filename="file:///$(find fra333_lab4_01_description)/mesh/link_0.STL"/>
             </geometry>
         </visual>
@@ -12,5 +12,5 @@
             <contact_coefficients mu="0" kp="1000.0" kd="1.0"/>
             <geometry>
-                <mesh filename="file:///$(find fra333_lab3_01_description)/mesh/link_0.STL"/>
+                <mesh filename="file:///$(find fra333_lab4_01_description)/mesh/link_0.STL"/>
             </geometry>
         </collision>
@@ -24,5 +24,5 @@
         <visual>
             <geometry>
-                <mesh filename="file:///$(find fra333_lab3_01_description)/mesh/link_1.STL"/>
+                <mesh filename="file:///$(find fra333_lab4_01_description)/mesh/link_1.STL"/>
             </geometry>
         </visual>
@@ -30,5 +30,5 @@
             <contact_coefficients mu="0" kp="1000.0" kd="1.0"/>
             <geometry>
-                <mesh filename="file:///$(find fra333_lab3_01_description)/mesh/link_1.STL"/>
+                <mesh filename="file:///$(find fra333_lab4_01_description)/mesh/link_1.STL"/>
             </geometry>
         </collision>
@@ -42,5 +42,5 @@
         <visual>
             <geometry>
-                <mesh filename="file:///$(find fra333_lab3_01_description)/mesh/link_2.STL"/>
+                <mesh filename="file:///$(find fra333_lab4_01_description)/mesh/link_2.STL"/>
             </geometry>
         </visual>
@@ -48,5 +48,5 @@
             <contact_coefficients mu="0" kp="1000.0" kd="1.0"/>
             <geometry>
-                <mesh filename="file:///$(find fra333_lab3_01_description)/mesh/link_2.STL"/>
+                <mesh filename="file:///$(find fra333_lab4_01_description)/mesh/link_2.STL"/>
             </geometry>
         </collision>
@@ -60,5 +60,5 @@
         <visual>
             <geometry>
-                <mesh filename="file:///$(find fra333_lab3_01_description)/mesh/link_3.STL"/>
+                <mesh filename="file:///$(find fra333_lab4_01_description)/mesh/link_3.STL"/>
             </geometry>
         </visual>
@@ -66,5 +66,5 @@
             <contact_coefficients mu="0" kp="1000.0" kd="1.0"/>
             <geometry>
-                <mesh filename="file:///$(find fra333_lab3_01_description)/mesh/link_3.STL"/>
+                <mesh filename="file:///$(find fra333_lab4_01_description)/mesh/link_3.STL"/>
             </geometry>
         </collision>
@@ -78,5 +78,5 @@
         <visual>
             <geometry>
-                <mesh filename="file:///$(find fra333_lab3_01_description)/mesh/gripper.STL"/>
+                <mesh filename="file:///$(find fra333_lab4_01_description)/mesh/gripper.STL"/>
             </geometry>
         </visual>
@@ -84,5 +84,5 @@
             <contact_coefficients mu="0" kp="1000.0" kd="1.0"/>
             <geometry>
-                <mesh filename="file:///$(find fra333_lab3_01_description)/mesh/gripper.STL"/>
+                <mesh filename="file:///$(find fra333_lab4_01_description)/mesh/gripper.STL"/>
             </geometry>
         </collision>
