Commit message: add scheduler

File: fra333_lab4_01/fra333_lab4_01_description/robot/sentinel.urdf.xacro (robot description, xacro)
@@ -3,4 +3,23 @@
     <!-- add more codes -->
     <link name="world"></link>
+    <link name="base_link">
+        <visual>
+        <origin xyz="0.0 0.0 0.005"/>
+            <geometry>
+                <mesh filename="file:///$(find fra333_lab4_01_description)/mesh/base_link.STL"/>
+            </geometry>
+        </visual>
+        <collision>
+            <contact_coefficients mu="0" kp="1000.0" kd="1.0"/>
+            <geometry>
+                <mesh filename="file:///$(find fra333_lab4_01_description)/mesh/base_link.STL"/>
+            </geometry>
+        </collision>
+        <inertial>
+            <origin xyz="0.0 0.0 0.0" rpy="0.0 0.0 0.0"/>
+            <mass value="1.0"/>
+            <inertia ixx="0.0003890077" ixy="0.0" ixz="0.0" iyy="0.0003890077" iyz="0.0" izz="0.0005310862"/>
+        </inertial>
+    </link>
     <link name="link_0">
         <visual>
@@ -93,6 +112,11 @@
         </inertial>
     </link>
-    <joint name="base_to_link_0" type="fixed">
+    <joint name="base_link_to_world" type="fixed">
        <parent link="world"/>
+       <child link="base_link"/>
+       <origin xyz="0.0 0.0 0.035"/>
+     </joint>
+     <joint name="base_to_link_0" type="fixed">
+       <parent link="base_link"/>
        <child link="link_0"/>
        <origin xyz="0.0 0.0 0.035"/>

Commit message: fix IK&scheduler

File: fra333_lab4_01/fra333_lab4_01_description/robot/sentinel.urdf.xacro (robot description, xacro)
@@ -11,5 +11,5 @@
         </visual>
         <collision>
-            <contact_coefficients mu="0" kp="1000.0" kd="1.0"/>
+            <contact_coefficients mu="0" kp="1.0" kd="1.0"/>
             <geometry>
                 <mesh filename="file:///$(find fra333_lab4_01_description)/mesh/base_link.STL"/>
@@ -29,5 +29,5 @@
         </visual>
         <collision>
-            <contact_coefficients mu="0" kp="1000.0" kd="1.0"/>
+            <contact_coefficients mu="0" kp="1.0" kd="1.0"/>
             <geometry>
                 <mesh filename="file:///$(find fra333_lab4_01_description)/mesh/link_0.STL"/>
@@ -47,5 +47,5 @@
         </visual>
         <collision>
-            <contact_coefficients mu="0" kp="1000.0" kd="1.0"/>
+            <contact_coefficients mu="0" kp="1.0" kd="1.0"/>
             <geometry>
                 <mesh filename="file:///$(find fra333_lab4_01_description)/mesh/link_1.STL"/>
@@ -65,5 +65,5 @@
         </visual>
         <collision>
-            <contact_coefficients mu="0" kp="1000.0" kd="1.0"/>
+            <contact_coefficients mu="0" kp="1.0" kd="1.0"/>
             <geometry>
                 <mesh filename="file:///$(find fra333_lab4_01_description)/mesh/link_2.STL"/>
@@ -83,5 +83,5 @@
         </visual>
         <collision>
-            <contact_coefficients mu="0" kp="1000.0" kd="1.0"/>
+            <contact_coefficients mu="0" kp="1.0" kd="1.0"/>
             <geometry>
                 <mesh filename="file:///$(find fra333_lab4_01_description)/mesh/link_3.STL"/>
@@ -101,5 +101,5 @@
         </visual>
         <collision>
-            <contact_coefficients mu="0" kp="1000.0" kd="1.0"/>
+            <contact_coefficients mu="0" kp="1.0" kd="1.0"/>
             <geometry>
                 <mesh filename="file:///$(find fra333_lab4_01_description)/mesh/gripper.STL"/>
@@ -108,5 +108,5 @@
         <inertial>
             <origin xyz="0.0 0.0 0.0" rpy="0.0 0.0 0.0"/>
-            <mass value="8.945"/>
+            <mass value="0.8945"/>
             <inertia ixx="0.0000831101" ixy="0.0" ixz="0.0" iyy="0.0081156101" iyz="0.0" izz="0.00005080097"/>
         </inertial>
@@ -128,5 +128,5 @@
        <axis xyz="0.0 0.0 1.0"/>
        <limit lower="-3" upper="3" effort="100.0" velocity="1.0"/>
-       <dynamics damping="0.1" friction="0.1"/>
+       <dynamics damping="10.0" friction="10.0"/>
      </joint>
      <joint name="link_1_to_2" type="revolute">
@@ -136,5 +136,5 @@
        <axis xyz="0.0 0.0 1.0"/>
        <limit lower="0" upper="3" effort="100.0" velocity="1.0"/>
-       <dynamics damping="0.1" friction="0.1"/>
+       <dynamics damping="10.0" friction="10.0"/>
      </joint>
      <joint name="link_2_to_3" type="revolute">
@@ -144,5 +144,5 @@
        <axis xyz="0.0 0.0 1.0"/>
        <limit lower="-2" upper="2" effort="100.0" velocity="1.0"/>
-       <dynamics damping="0.1" friction="0.1"/>
+       <dynamics damping="10.0" friction="10.0"/>
      </joint>
     <joint name="link_3_to_gripper" type="fixed">
